Commit message: Update description_omni_robot.urdf

File: urdf/description_omni_robot.urdf (robot description, URDF)
Before this commit: robot description_omni_robot, 9 links, 8 joints
Links:
- link camera_link: geometry collision mesh filename=package://description_omni/meshes/camera_link.STL; visual mesh filename=package://description_omni/meshes/camera_link.STL
Joints:
- joint camera_joint: origin xyz=0.0712462120245874 -0.00019894784923466 0.0677413009524857 rpy=0 0 0 -> xyz=0.0712462120245874 -0.00019894784923466 0.0677413009524857 rpy=-1.5707963267949 0 -1.5707963267949

Commit message: Update description_omni_robot.urdf

File: urdf/description_omni_robot.urdf (robot description, URDF)
Before this commit: robot description_omni_robot, 9 links, 8 joints
Links:
- link camera_link: geometry collision mesh filename=package://description_omni_robot/meshes/camera_link.STL; visual mesh filename=package://description_omni_robot/meshes/camera_link.STL
Joints:
- joint camera_joint: origin xyz=0.0712462120245874 -0.00019894784923466 0.0677413009524857 rpy=-1.5707963267949 0 -1.5707963267949 -> xyz=0.0712462120245874 -0.00019894784923466 0.0677413009524857 rpy=0 0 0

Commit message: new

File: urdf/description_omni_robot.urdf (robot description, URDF)
Before this commit: robot description_omni_robot, 9 links, 8 joints
Joints:
- joint arm_1_joint: limit lower=-1.57 upper=1.57 effort=300 velocity=10 -> lower=-1.5707963267949 upper=1.5707963267949 effort=100 velocity=10
- joint arm_2_joint: limit lower=-1.57 upper=1.57 effort=300 velocity=10 -> lower=-1.5707963267949 upper=1.5707963267949 effort=100 velocity=10
